Commit message: Deteccion de texto implementando movimiento

File: retos_ws/src/simulador_gazebo/models/Cybercrex_frontal/camera.xacro (robot description, xacro)
@@ -4,5 +4,5 @@
         <parent link="chassis"/>
         <child link="camera_link"/>
-        <origin xyz="0.257 0 1.165" rpy="0 0.610865 0"/>
+        <origin xyz="0.257 0 0.465" rpy="0 0.610865 0"/>
     </joint>
     <link name="camera_link">

Commit message: Actualizacion del programa deteccion de texto

File: retos_ws/src/simulador_gazebo/models/Cybercrex_frontal/camera.xacro (robot description, xacro)
@@ -4,5 +4,5 @@
         <parent link="chassis"/>
         <child link="camera_link"/>
-        <origin xyz="0.257 0 0.465" rpy="0 0.610865 0"/>
+        <origin xyz="0.257 0 1.0" rpy="0 ${pi/5} 0"/>
     </joint>
     <link name="camera_link">
